File: smarkant-kicad/smarkant.sch (KiCad schematic (older format))
At the start: 30 parts, among them IC1 ATMEGA328P-P, P1 POW24V, P2 UP, P3 DOWN, P4 ISP, P5 SERIAL1, P6 LINBUS, P7 SERIAL2, Q1 2N3904, SW1 D9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

Commit message: fix: power rail is 3.3V instead of 5V
Connections:
- net labels added: +3.3V
Changed lines of the file:
@@
-$EndComp
-$Comp
-L +5V #PWR1
-U 1 1 588E6F4A
-P 1050 950
-F 0 "#PWR1" H 1050 800 50  0001 C CNN
-F 1 "+5V" H 1050 1090 50  0000 C CNN
-F 2 "" H 1050 950 50  0000 C CNN
-F 3 "" H 1050 950 50  0000 C CNN
-	1    1050 950
-	1    0    0    -1
 $EndComp
 $Comp
@@
 $EndComp
 $Comp
-L +5V #PWR7
-U 1 1 588F4860
-P 3500 6100
-F 0 "#PWR7" H 3500 5950 50  0001 C CNN
-F 1 "+5V" H 3500 6240 50  0000 C CNN
-F 2 "" H 3500 6100 50  0000 C CNN
-F 3 "" H 3500 6100 50  0000 C CNN
-	1    3500 6100
-	1    0    0    -1
-$EndComp
-$Comp
 L BC547 Q1
 U 1 1 588FA8DF
@@
 $EndComp
 $Comp
-L +5V #PWR14
-U 1 1 588FE413
-P 5700 4150
-F 0 "#PWR14" H 5700 4000 50  0001 C CNN
-F 1 "+5V" H 5700 4290 50  0000 C CNN
-F 2 "" H 5700 4150 50  0000 C CNN
-F 3 "" H 5700 4150 50  0000 C CNN
-	1    5700 4150
-	-1   0    0    -1
-$EndComp
-$Comp
 L ATMEGA328P-P IC1
 U 1 1 58BAD282
@@
 $EndComp
 $Comp
-L +5V #PWR10
-U 1 1 58BB6260
-P 4700 4850
-F 0 "#PWR10" H 4700 4700 50  0001 C CNN
-F 1 "+5V" H 4700 4990 50  0000 C CNN
-F 2 "" H 4700 4850 50  0000 C CNN
-F 3 "" H 4700 4850 50  0000 C CNN
-	1    4700 4850
-	1    0    0    -1
-$EndComp
-$Comp
-L +5V #PWR12
-U 1 1 58BB7DB8
-P 4750 2650
-F 0 "#PWR12" H 4750 2500 50  0001 C CNN
-F 1 "+5V" H 4750 2790 50  0000 C CNN
-F 2 "" H 4750 2650 50  0000 C CNN
-F 3 "" H 4750 2650 50  0000 C CNN
-	1    4750 2650
-	0    1    1    0
-$EndComp
-$Comp
 L ESP-12E U2
 U 1 1 58BBA5F5
@@
 Wire Wire Line
 	10500 1400 10500 5300
-$Comp
-L +5V #PWR25
-U 1 1 58BC2377
-P 10500 1000
-F 0 "#PWR25" H 10500 850 50  0001 C CNN
-F 1 "+5V" H 10500 1140 50  0000 C CNN
-F 2 "" H 10500 1000 50  0000 C CNN
-F 3 "" H 10500 1000 50  0000 C CNN
-	1    10500 1000
-	-1   0    0    -1
-$EndComp
 Connection ~ 10500 2800
 Wire Wire Line
@@
 	1    0    0    1
 $EndComp
-$Comp
-L +5V #PWR19
-U 1 1 58BD59B6
-P 7900 950
-F 0 "#PWR19" H 7900 800 50  0001 C CNN
-F 1 "+5V" H 7900 1090 50  0000 C CNN
-F 2 "" H 7900 950 50  0000 C CNN
-F 3 "" H 7900 950 50  0000 C CNN
-	1    7900 950
-	-1   0    0    -1
-$EndComp
 Wire Wire Line
 	7900 950  7900 1100
@@
 	1    0    0    1
 $EndComp
-$Comp
-L +5V #PWR17
-U 1 1 58BD773F
+Wire Wire Line
+	7750 950  7750 1100
+Wire Wire Line
+	8050 2600 7750 2600
+Wire Wire Line
+	7750 2600 7750 1400
+Wire Wire Line
+	10200 1550 10200 2700
+Wire Wire Line
+	10000 1750 10000 2600
+$Comp
+L +3.3V #PWR?
+U 1 1 58D085AB
+P 3500 6100
+F 0 "#PWR?" H 3500 5950 50  0001 C CNN
+F 1 "+3.3V" H 3500 6240 50  0000 C CNN
+F 2 "" H 3500 6100 50  0000 C CNN
+F 3 "" H 3500 6100 50  0000 C CNN
+	1    3500 6100
+	1    0    0    -1
+$EndComp
+$Comp
+L +3.3V #PWR?
+U 1 1 58D086D2
+P 4700 4850
+F 0 "#PWR?" H 4700 4700 50  0001 C CNN
+F 1 "+3.3V" H 4700 4990 50  0000 C CNN
+F 2 "" H 4700 4850 50  0000 C CNN
+F 3 "" H 4700 4850 50  0000 C CNN
+	1    4700 4850
+	1    0    0    -1
+$EndComp
+$Comp
+L +3.3V #PWR?
+U 1 1 58D08E80
+P 5700 4150
+F 0 "#PWR?" H 5700 4000 50  0001 C CNN
+F 1 "+3.3V" H 5700 4290 50  0000 C CNN
+F 2 "" H 5700 4150 50  0000 C CNN
+F 3 "" H 5700 4150 50  0000 C CNN
+	1    5700 4150
+	1    0    0    -1
+$EndComp
+$Comp
+L +3.3V #PWR?
+U 1 1 58D09C86
+P 1050 950
+F 0 "#PWR?" H 1050 800 50  0001 C CNN
+F 1 "+3.3V" H 1050 1090 50  0000 C CNN
+F 2 "" H 1050 950 50  0000 C CNN
+F 3 "" H 1050 950 50  0000 C CNN
+	1    1050 950
+	1    0    0    -1
+$EndComp
+$Comp
+L +3.3V #PWR?
+U 1 1 58D0A56A
 P 7750 950
-F 0 "#PWR17" H 7750 800 50  0001 C CNN
-F 1 "+5V" H 7750 1090 50  0000 C CNN
+F 0 "#PWR?" H 7750 800 50  0001 C CNN
+F 1 "+3.3V" H 7750 1090 50  0000 C CNN
 F 2 "" H 7750 950 50  0000 C CNN
 F 3 "" H 7750 950 50  0000 C CNN
 	1    7750 950
-	-1   0    0    -1
-$EndComp
-Wire Wire Line
-	7750 950  7750 1100
-Wire Wire Line
-	8050 2600 7750 2600
-Wire Wire Line
-	7750 2600 7750 1400
-Wire Wire Line
-	10200 1550 10200 2700
-Wire Wire Line
-	10000 1750 10000 2600
+	1    0    0    -1
+$EndComp
+$Comp
+L +3.3V #PWR?
+U 1 1 58D0A606
+P 7900 950
+F 0 "#PWR?" H 7900 800 50  0001 C CNN
+F 1 "+3.3V" H 7900 1090 50  0000 C CNN
+F 2 "" H 7900 950 50  0000 C CNN
+F 3 "" H 7900 950 50  0000 C CNN
+	1    7900 950
+	1    0    0    -1
+$EndComp
+$Comp
+L +3.3V #PWR?
+U 1 1 58D0A668
+P 10500 1000
+F 0 "#PWR?" H 10500 850 50  0001 C CNN
+F 1 "+3.3V" H 10500 1140 50  0000 C CNN
+F 2 "" H 10500 1000 50  0000 C CNN
+F 3 "" H 10500 1000 50  0000 C CNN
+	1    10500 1000
+	1    0    0    -1
+$EndComp
+$Comp
+L +3.3V #PWR?
+U 1 1 58D0B015
+P 4750 2650
+F 0 "#PWR?" H 4750 2500 50  0001 C CNN
+F 1 "+3.3V" H 4750 2790 50  0000 C CNN
+F 2 "" H 4750 2650 50  0000 C CNN
+F 3 "" H 4750 2650 50  0000 C CNN
+	1    4750 2650
+	0    1    1    0
+$EndComp
 $EndSCHEMATC
